File: LED_Part10.sch (KiCad schematic (older format))
At the start: 13 parts

Commit message: Ruan: modify LED part
Parts:
- gave numbers to parts that had none: 13
Changed lines of the file:
@@
 AR Path="/5DF7BF4B/5E039D16" Ref="R?"  Part="1"
 AR Path="/5DFD1EC3/5E039D16" Ref="R?"  Part="1"
-AR Path="/5E02C61B/5E039D16" Ref="R?"  Part="1"
+AR Path="/5E02C61B/5E039D16" Ref="R33"  Part="1"
 AR Path="/5E08B2E9/5E039D16" Ref="R?"  Part="1"
 AR Path="/5E0EDFEE/5E039D16" Ref="R?"  Part="1"
-F 0 "R?" V 7493 3500 50  0000 C CNN
+F 0 "R33" V 7493 3500 50  0000 C CNN
 F 1 "10K" V 7584 3500 50  0000 C CNN
 F 2 "Resistor_SMD:R_0603_1608Metric" V 7630 3500 50  0001 C CNN
@@
 AR Path="/5DF7BF4B/5E039D4D" Ref="U?"  Part="1"
 AR Path="/5DFD1EC3/5E039D4D" Ref="U?"  Part="1"
-AR Path="/5E02C61B/5E039D4D" Ref="U?"  Part="1"
+AR Path="/5E02C61B/5E039D4D" Ref="U26"  Part="1"
 AR Path="/5E08B2E9/5E039D4D" Ref="U?"  Part="1"
 AR Path="/5E0EDFEE/5E039D4D" Ref="U?"  Part="1"
-F 0 "U?" H 3700 4415 50  0000 C CNN
+F 0 "U26" H 3700 4415 50  0000 C CNN
 F 1 "TCS3200" H 3700 4324 50  0000 C CNN
 F 2 "Package_SO:SOIC-8_3.9x4.9mm_P1.27mm" H 3600 4150 50  0001 C CNN
@@
 AR Path="/5DF7BF4B/5E039D53" Ref="C?"  Part="1"
 AR Path="/5DFD1EC3/5E039D53" Ref="C?"  Part="1"
-AR Path="/5E02C61B/5E039D53" Ref="C?"  Part="1"
+AR Path="/5E02C61B/5E039D53" Ref="C82"  Part="1"
 AR Path="/5E08B2E9/5E039D53" Ref="C?"  Part="1"
 AR Path="/5E0EDFEE/5E039D53" Ref="C?"  Part="1"
-F 0 "C?" H 3935 5004 50  0000 R CNN
+F 0 "C82" H 3935 5004 50  0000 R CNN
 F 1 "0.1uF" H 3935 5095 50  0000 R CNN
 F 2 "Capacitor_SMD:C_0603_1608Metric" H 4088 4900 50  0001 C CNN
@@
 AR Path="/5DF7BF4B/5E039D59" Ref="C?"  Part="1"
 AR Path="/5DFD1EC3/5E039D59" Ref="C?"  Part="1"
-AR Path="/5E02C61B/5E039D59" Ref="C?"  Part="1"
+AR Path="/5E02C61B/5E039D59" Ref="C81"  Part="1"
 AR Path="/5E08B2E9/5E039D59" Ref="C?"  Part="1"
 AR Path="/5E0EDFEE/5E039D59" Ref="C?"  Part="1"
-F 0 "C?" V 3352 3350 50  0000 C CNN
+F 0 "C81" V 3352 3350 50  0000 C CNN
 F 1 "20pF" V 3261 3350 50  0000 C CNN
 F 2 "Capacitor_SMD:C_0603_1608Metric" H 3138 3200 50  0001 C CNN
@@
 AR Path="/5DF7BF4B/5E039D5F" Ref="C?"  Part="1"
 AR Path="/5DFD1EC3/5E039D5F" Ref="C?"  Part="1"
-AR Path="/5E02C61B/5E039D5F" Ref="C?"  Part="1"
+AR Path="/5E02C61B/5E039D5F" Ref="C80"  Part="1"
 AR Path="/5E08B2E9/5E039D5F" Ref="C?"  Part="1"
 AR Path="/5E0EDFEE/5E039D5F" Ref="C?"  Part="1"
-F 0 "C?" V 3352 3000 50  0000 C CNN
+F 0 "C80" V 3352 3000 50  0000 C CNN
 F 1 "20pF" V 3261 3000 50  0000 C CNN
 F 2 "Capacitor_SMD:C_0603_1608Metric" H 3138 2850 50  0001 C CNN
@@
 AR Path="/5DF7BF4B/5E039D65" Ref="C?"  Part="1"
 AR Path="/5DFD1EC3/5E039D65" Ref="C?"  Part="1"
-AR Path="/5E02C61B/5E039D65" Ref="C?"  Part="1"
+AR Path="/5E02C61B/5E039D65" Ref="C86"  Part="1"
 AR Path="/5E08B2E9/5E039D65" Ref="C?"  Part="1"
 AR Path="/5E0EDFEE/5E039D65" Ref="C?"  Part="1"
-F 0 "C?" H 6635 2304 50  0000 R CNN
+F 0 "C86" H 6635 2304 50  0000 R CNN
 F 1 "0.1uF" H 6635 2395 50  0000 R CNN
 F 2 "Capacitor_SMD:C_0603_1608Metric" H 6788 2200 50  0001 C CNN
@@
 AR Path="/5DF7BF4B/5E039D6D" Ref="C?"  Part="1"
 AR Path="/5DFD1EC3/5E039D6D" Ref="C?"  Part="1"
-AR Path="/5E02C61B/5E039D6D" Ref="C?"  Part="1"
+AR Path="/5E02C61B/5E039D6D" Ref="C85"  Part="1"
 AR Path="/5E08B2E9/5E039D6D" Ref="C?"  Part="1"
 AR Path="/5E0EDFEE/5E039D6D" Ref="C?"  Part="1"
-F 0 "C?" H 6335 2304 50  0000 R CNN
+F 0 "C85" H 6335 2304 50  0000 R CNN
 F 1 "0.1uF" H 6335 2395 50  0000 R CNN
 F 2 "Capacitor_SMD:C_0603_1608Metric" H 6488 2200 50  0001 C CNN
@@
 AR Path="/5DF7BF4B/5E039D79" Ref="#PWR?"  Part="1"
 AR Path="/5DFD1EC3/5E039D79" Ref="#PWR?"  Part="1"
-AR Path="/5E02C61B/5E039D79" Ref="#PWR?"  Part="1"
+AR Path="/5E02C61B/5E039D79" Ref="#PWR091"  Part="1"
 AR Path="/5E08B2E9/5E039D79" Ref="#PWR?"  Part="1"
 AR Path="/5E0EDFEE/5E039D79" Ref="#PWR?"  Part="1"
-F 0 "#PWR?" H 6300 2450 50  0001 C CNN
+F 0 "#PWR091" H 6300 2450 50  0001 C CNN
 F 1 "GND" H 6305 2527 50  0000 C CNN
 F 2 "" H 6300 2700 50  0001 C CNN
@@
 AR Path="/5DF7BF4B/5E039D7F" Ref="C?"  Part="1"
 AR Path="/5DFD1EC3/5E039D7F" Ref="C?"  Part="1"
-AR Path="/5E02C61B/5E039D7F" Ref="C?"  Part="1"
+AR Path="/5E02C61B/5E039D7F" Ref="C84"  Part="1"
 AR Path="/5E08B2E9/5E039D7F" Ref="C?"  Part="1"
 AR Path="/5E0EDFEE/5E039D7F" Ref="C?"  Part="1"
-F 0 "C?" H 6035 2304 50  0000 R CNN
+F 0 "C84" H 6035 2304 50  0000 R CNN
 F 1 "0.1uF" H 6035 2395 50  0000 R CNN
 F 2 "Capacitor_SMD:C_0603_1608Metric" H 6188 2200 50  0001 C CNN
@@
 AR Path="/5DF7BF4B/5E039D85" Ref="C?"  Part="1"
 AR Path="/5DFD1EC3/5E039D85" Ref="C?"  Part="1"
-AR Path="/5E02C61B/5E039D85" Ref="C?"  Part="1"
+AR Path="/5E02C61B/5E039D85" Ref="C83"  Part="1"
 AR Path="/5E08B2E9/5E039D85" Ref="C?"  Part="1"
 AR Path="/5E0EDFEE/5E039D85" Ref="C?"  Part="1"
-F 0 "C?" H 5735 2304 50  0000 R CNN
+F 0 "C83" H 5735 2304 50  0000 R CNN
 F 1 "1uF" H 5735 2395 50  0000 R CNN
 F 2 "Capacitor_SMD:C_0603_1608Metric" H 5888 2200 50  0001 C CNN
@@
 AR Path="/5DF7BF4B/5E039D8B" Ref="#PWR?"  Part="1"
 AR Path="/5DFD1EC3/5E039D8B" Ref="#PWR?"  Part="1"
-AR Path="/5E02C61B/5E039D8B" Ref="#PWR?"  Part="1"
+AR Path="/5E02C61B/5E039D8B" Ref="#PWR090"  Part="1"
 AR Path="/5E08B2E9/5E039D8B" Ref="#PWR?"  Part="1"
 AR Path="/5E0EDFEE/5E039D8B" Ref="#PWR?"  Part="1"
-F 0 "#PWR?" H 6200 4250 50  0001 C CNN
+F 0 "#PWR090" H 6200 4250 50  0001 C CNN
 F 1 "GND" H 6205 4327 50  0000 C CNN
 F 2 "" H 6200 4500 50  0001 C CNN
@@
 AR Path="/5DF7BF4B/5E039D91" Ref="#PWR?"  Part="1"
 AR Path="/5DFD1EC3/5E039D91" Ref="#PWR?"  Part="1"
-AR Path="/5E02C61B/5E039D91" Ref="#PWR?"  Part="1"
+AR Path="/5E02C61B/5E039D91" Ref="#PWR088"  Part="1"
 AR Path="/5E08B2E9/5E039D91" Ref="#PWR?"  Part="1"
 AR Path="/5E0EDFEE/5E039D91" Ref="#PWR?"  Part="1"
-F 0 "#PWR?" H 4050 4950 50  0001 C CNN
+F 0 "#PWR088" H 4050 4950 50  0001 C CNN
 F 1 "GND" H 4055 5027 50  0000 C CNN
 F 2 "" H 4050 5200 50  0001 C CNN
@@
 AR Path="/5DF7BF4B/5E039DAD" Ref="#PWR?"  Part="1"
 AR Path="/5DFD1EC3/5E039DAD" Ref="#PWR?"  Part="1"
-AR Path="/5E02C61B/5E039DAD" Ref="#PWR?"  Part="1"
+AR Path="/5E02C61B/5E039DAD" Ref="#PWR089"  Part="1"
 AR Path="/5E08B2E9/5E039DAD" Ref="#PWR?"  Part="1"
 AR Path="/5E0EDFEE/5E039DAD" Ref="#PWR?"  Part="1"
-F 0 "#PWR?" H 5600 4900 50  0001 C CNN
+F 0 "#PWR089" H 5600 4900 50  0001 C CNN
 F 1 "GND" H 5605 4977 50  0000 C CNN
 F 2 "" H 5600 5150 50  0001 C CNN
@@
 AR Path="/5DF7BF4B/5E039DC3" Ref="#PWR?"  Part="1"
 AR Path="/5DFD1EC3/5E039DC3" Ref="#PWR?"  Part="1"
-AR Path="/5E02C61B/5E039DC3" Ref="#PWR?"  Part="1"
+AR Path="/5E02C61B/5E039DC3" Ref="#PWR085"  Part="1"
 AR Path="/5E08B2E9/5E039DC3" Ref="#PWR?"  Part="1"
 AR Path="/5E0EDFEE/5E039DC3" Ref="#PWR?"  Part="1"
-F 0 "#PWR?" H 2700 3200 50  0001 C CNN
+F 0 "#PWR085" H 2700 3200 50  0001 C CNN
 F 1 "GND" H 2705 3277 50  0000 C CNN
 F 2 "" H 2700 3450 50  0001 C CNN
@@
 AR Path="/5DF7BF4B/5E039DD2" Ref="Y?"  Part="1"
 AR Path="/5DFD1EC3/5E039DD2" Ref="Y?"  Part="1"
-AR Path="/5E02C61B/5E039DD2" Ref="Y?"  Part="1"
+AR Path="/5E02C61B/5E039DD2" Ref="Y11"  Part="1"
 AR Path="/5E08B2E9/5E039DD2" Ref="Y?"  Part="1"
 AR Path="/5E0EDFEE/5E039DD2" Ref="Y?"  Part="1"
-F 0 "Y?" V 3604 3331 50  0000 L CNN
+F 0 "Y11" V 3604 3331 50  0000 L CNN
 F 1 "8MHz" V 3695 3331 50  0000 L CNN
 F 2 "Crystal:Crystal_SMD_3225-4Pin_3.2x2.5mm_HandSoldering" H 3650 3200 50  0001 C CNN
@@
 AR Path="/5DF7BF4B/5E039DDA" Ref="R?"  Part="1"
 AR Path="/5DFD1EC3/5E039DDA" Ref="R?"  Part="1"
-AR Path="/5E02C61B/5E039DDA" Ref="R?"  Part="1"
+AR Path="/5E02C61B/5E039DDA" Ref="R32"  Part="1"
 AR Path="/5E08B2E9/5E039DDA" Ref="R?"  Part="1"
 AR Path="/5E0EDFEE/5E039DDA" Ref="R?"  Part="1"
-F 0 "R?" V 3993 2350 50  0000 C CNN
+F 0 "R32" V 3993 2350 50  0000 C CNN
 F 1 "10K" V 4084 2350 50  0000 C CNN
 F 2 "Resistor_SMD:R_0603_1608Metric" V 4130 2350 50  0001 C CNN
@@
 AR Path="/5DF7BF4B/5E039DE1" Ref="#PWR?"  Part="1"
 AR Path="/5DFD1EC3/5E039DE1" Ref="#PWR?"  Part="1"
-AR Path="/5E02C61B/5E039DE1" Ref="#PWR?"  Part="1"
+AR Path="/5E02C61B/5E039DE1" Ref="#PWR087"  Part="1"
 AR Path="/5E08B2E9/5E039DE1" Ref="#PWR?"  Part="1"
 AR Path="/5E0EDFEE/5E039DE1" Ref="#PWR?"  Part="1"
-F 0 "#PWR?" H 3900 2300 50  0001 C CNN
+F 0 "#PWR087" H 3900 2300 50  0001 C CNN
 F 1 "GND" H 3905 2377 50  0000 C CNN
 F 2 "" H 3900 2550 50  0001 C CNN
@@
 AR Path="/5DF7BF4B/5E039DE7" Ref="#PWR?"  Part="1"
 AR Path="/5DFD1EC3/5E039DE7" Ref="#PWR?"  Part="1"
-AR Path="/5E02C61B/5E039DE7" Ref="#PWR?"  Part="1"
+AR Path="/5E02C61B/5E039DE7" Ref="#PWR086"  Part="1"
 AR Path="/5E08B2E9/5E039DE7" Ref="#PWR?"  Part="1"
 AR Path="/5E0EDFEE/5E039DE7" Ref="#PWR?"  Part="1"
-F 0 "#PWR?" H 3100 4350 50  0001 C CNN
+F 0 "#PWR086" H 3100 4350 50  0001 C CNN
 F 1 "GND" H 3105 4427 50  0000 C CNN
 F 2 "" H 3100 4600 50  0001 C CNN
@@
 AR Path="/5DF7BF4B/5E039DF0" Ref="U?"  Part="1"
 AR Path="/5DFD1EC3/5E039DF0" Ref="U?"  Part="1"
-AR Path="/5E02C61B/5E039DF0" Ref="U?"  Part="1"
+AR Path="/5E02C61B/5E039DF0" Ref="U27"  Part="1"
 AR Path="/5E08B2E9/5E039DF0" Ref="U?"  Part="1"
 AR Path="/5E0EDFEE/5E039DF0" Ref="U?"  Part="1"
-F 0 "U?" H 5150 2061 50  0000 C CNN
+F 0 "U27" H 5150 2061 50  0000 C CNN
 F 1 "STM32F103C8T6" H 5150 1970 50  0000 C CNN
 F 2 "Package_QFP:LQFP-48_7x7mm_P0.5mm" H 4600 2250 50  0001 R CNN
@@
 AR Path="/5E039E03" Ref="J?"  Part="1"
 AR Path="/5E0EDFEE/5E039E03" Ref="J?"  Part="1"
-F 0 "J?" H 6480 4792 50  0000 L CNN
+AR Path="/5E02C61B/5E039E03" Ref="J11"  Part="1"
+F 0 "J11" H 6480 4792 50  0000 L CNN
 F 1 "Conn_01x03" H 6480 4701 50  0000 L CNN
 F 2 "RuanProject:Connector_Set_1x03_P2.54mm_Vertical" H 6400 4750 50  0001 C CNN
