File: LED_Part11.sch (KiCad schematic (older format))
At the start: 13 parts

Commit message: Ruan: modify LED part
Parts:
- gave numbers to parts that had none: 13
Changed lines of the file:
@@
 AR Path="/5DFD1EC3/5E0342E7" Ref="R?"  Part="1"
 AR Path="/5E02C61B/5E0342E7" Ref="R?"  Part="1"
-AR Path="/5E08B2E9/5E0342E7" Ref="R?"  Part="1"
+AR Path="/5E08B2E9/5E0342E7" Ref="R35"  Part="1"
 AR Path="/5E0EDFEE/5E0342E7" Ref="R?"  Part="1"
-F 0 "R?" V 7793 3750 50  0000 C CNN
+F 0 "R35" V 7793 3750 50  0000 C CNN
 F 1 "10K" V 7884 3750 50  0000 C CNN
 F 2 "Resistor_SMD:R_0603_1608Metric" V 7930 3750 50  0001 C CNN
@@
 AR Path="/5DFD1EC3/5E03431E" Ref="U?"  Part="1"
 AR Path="/5E02C61B/5E03431E" Ref="U?"  Part="1"
-AR Path="/5E08B2E9/5E03431E" Ref="U?"  Part="1"
+AR Path="/5E08B2E9/5E03431E" Ref="U28"  Part="1"
 AR Path="/5E0EDFEE/5E03431E" Ref="U?"  Part="1"
-F 0 "U?" H 4000 4665 50  0000 C CNN
+F 0 "U28" H 4000 4665 50  0000 C CNN
 F 1 "TCS3200" H 4000 4574 50  0000 C CNN
 F 2 "Package_SO:SOIC-8_3.9x4.9mm_P1.27mm" H 3900 4400 50  0001 C CNN
@@
 AR Path="/5DFD1EC3/5E034324" Ref="C?"  Part="1"
 AR Path="/5E02C61B/5E034324" Ref="C?"  Part="1"
-AR Path="/5E08B2E9/5E034324" Ref="C?"  Part="1"
+AR Path="/5E08B2E9/5E034324" Ref="C89"  Part="1"
 AR Path="/5E0EDFEE/5E034324" Ref="C?"  Part="1"
-F 0 "C?" H 4235 5254 50  0000 R CNN
+F 0 "C89" H 4235 5254 50  0000 R CNN
 F 1 "0.1uF" H 4235 5345 50  0000 R CNN
 F 2 "Capacitor_SMD:C_0603_1608Metric" H 4388 5150 50  0001 C CNN
@@
 AR Path="/5DFD1EC3/5E03432A" Ref="C?"  Part="1"
 AR Path="/5E02C61B/5E03432A" Ref="C?"  Part="1"
-AR Path="/5E08B2E9/5E03432A" Ref="C?"  Part="1"
+AR Path="/5E08B2E9/5E03432A" Ref="C88"  Part="1"
 AR Path="/5E0EDFEE/5E03432A" Ref="C?"  Part="1"
-F 0 "C?" V 3652 3600 50  0000 C CNN
+F 0 "C88" V 3652 3600 50  0000 C CNN
 F 1 "20pF" V 3561 3600 50  0000 C CNN
 F 2 "Capacitor_SMD:C_0603_1608Metric" H 3438 3450 50  0001 C CNN
@@
 AR Path="/5DFD1EC3/5E034330" Ref="C?"  Part="1"
 AR Path="/5E02C61B/5E034330" Ref="C?"  Part="1"
-AR Path="/5E08B2E9/5E034330" Ref="C?"  Part="1"
+AR Path="/5E08B2E9/5E034330" Ref="C87"  Part="1"
 AR Path="/5E0EDFEE/5E034330" Ref="C?"  Part="1"
-F 0 "C?" V 3652 3250 50  0000 C CNN
+F 0 "C87" V 3652 3250 50  0000 C CNN
 F 1 "20pF" V 3561 3250 50  0000 C CNN
 F 2 "Capacitor_SMD:C_0603_1608Metric" H 3438 3100 50  0001 C CNN
@@
 AR Path="/5DFD1EC3/5E034336" Ref="C?"  Part="1"
 AR Path="/5E02C61B/5E034336" Ref="C?"  Part="1"
-AR Path="/5E08B2E9/5E034336" Ref="C?"  Part="1"
+AR Path="/5E08B2E9/5E034336" Ref="C93"  Part="1"
 AR Path="/5E0EDFEE/5E034336" Ref="C?"  Part="1"
-F 0 "C?" H 6935 2554 50  0000 R CNN
+F 0 "C93" H 6935 2554 50  0000 R CNN
 F 1 "0.1uF" H 6935 2645 50  0000 R CNN
 F 2 "Capacitor_SMD:C_0603_1608Metric" H 7088 2450 50  0001 C CNN
@@
 AR Path="/5DFD1EC3/5E03433E" Ref="C?"  Part="1"
 AR Path="/5E02C61B/5E03433E" Ref="C?"  Part="1"
-AR Path="/5E08B2E9/5E03433E" Ref="C?"  Part="1"
+AR Path="/5E08B2E9/5E03433E" Ref="C92"  Part="1"
 AR Path="/5E0EDFEE/5E03433E" Ref="C?"  Part="1"
-F 0 "C?" H 6635 2554 50  0000 R CNN
+F 0 "C92" H 6635 2554 50  0000 R CNN
 F 1 "0.1uF" H 6635 2645 50  0000 R CNN
 F 2 "Capacitor_SMD:C_0603_1608Metric" H 6788 2450 50  0001 C CNN
@@
 AR Path="/5DFD1EC3/5E03434A" Ref="#PWR?"  Part="1"
 AR Path="/5E02C61B/5E03434A" Ref="#PWR?"  Part="1"
-AR Path="/5E08B2E9/5E03434A" Ref="#PWR?"  Part="1"
+AR Path="/5E08B2E9/5E03434A" Ref="#PWR098"  Part="1"
 AR Path="/5E0EDFEE/5E03434A" Ref="#PWR?"  Part="1"
-F 0 "#PWR?" H 6600 2700 50  0001 C CNN
+F 0 "#PWR098" H 6600 2700 50  0001 C CNN
 F 1 "GND" H 6605 2777 50  0000 C CNN
 F 2 "" H 6600 2950 50  0001 C CNN
@@
 AR Path="/5DFD1EC3/5E034350" Ref="C?"  Part="1"
 AR Path="/5E02C61B/5E034350" Ref="C?"  Part="1"
-AR Path="/5E08B2E9/5E034350" Ref="C?"  Part="1"
+AR Path="/5E08B2E9/5E034350" Ref="C91"  Part="1"
 AR Path="/5E0EDFEE/5E034350" Ref="C?"  Part="1"
-F 0 "C?" H 6335 2554 50  0000 R CNN
+F 0 "C91" H 6335 2554 50  0000 R CNN
 F 1 "0.1uF" H 6335 2645 50  0000 R CNN
 F 2 "Capacitor_SMD:C_0603_1608Metric" H 6488 2450 50  0001 C CNN
@@
 AR Path="/5DFD1EC3/5E034356" Ref="C?"  Part="1"
 AR Path="/5E02C61B/5E034356" Ref="C?"  Part="1"
-AR Path="/5E08B2E9/5E034356" Ref="C?"  Part="1"
+AR Path="/5E08B2E9/5E034356" Ref="C90"  Part="1"
 AR Path="/5E0EDFEE/5E034356" Ref="C?"  Part="1"
-F 0 "C?" H 6035 2554 50  0000 R CNN
+F 0 "C90" H 6035 2554 50  0000 R CNN
 F 1 "1uF" H 6035 2645 50  0000 R CNN
 F 2 "Capacitor_SMD:C_0603_1608Metric" H 6188 2450 50  0001 C CNN
@@
 AR Path="/5DFD1EC3/5E03435C" Ref="#PWR?"  Part="1"
 AR Path="/5E02C61B/5E03435C" Ref="#PWR?"  Part="1"
-AR Path="/5E08B2E9/5E03435C" Ref="#PWR?"  Part="1"
+AR Path="/5E08B2E9/5E03435C" Ref="#PWR097"  Part="1"
 AR Path="/5E0EDFEE/5E03435C" Ref="#PWR?"  Part="1"
-F 0 "#PWR?" H 6500 4500 50  0001 C CNN
+F 0 "#PWR097" H 6500 4500 50  0001 C CNN
 F 1 "GND" H 6505 4577 50  0000 C CNN
 F 2 "" H 6500 4750 50  0001 C CNN
@@
 AR Path="/5DFD1EC3/5E034362" Ref="#PWR?"  Part="1"
 AR Path="/5E02C61B/5E034362" Ref="#PWR?"  Part="1"
-AR Path="/5E08B2E9/5E034362" Ref="#PWR?"  Part="1"
+AR Path="/5E08B2E9/5E034362" Ref="#PWR095"  Part="1"
 AR Path="/5E0EDFEE/5E034362" Ref="#PWR?"  Part="1"
-F 0 "#PWR?" H 4350 5200 50  0001 C CNN
+F 0 "#PWR095" H 4350 5200 50  0001 C CNN
 F 1 "GND" H 4355 5277 50  0000 C CNN
 F 2 "" H 4350 5450 50  0001 C CNN
@@
 AR Path="/5DFD1EC3/5E03437E" Ref="#PWR?"  Part="1"
 AR Path="/5E02C61B/5E03437E" Ref="#PWR?"  Part="1"
-AR Path="/5E08B2E9/5E03437E" Ref="#PWR?"  Part="1"
+AR Path="/5E08B2E9/5E03437E" Ref="#PWR096"  Part="1"
 AR Path="/5E0EDFEE/5E03437E" Ref="#PWR?"  Part="1"
-F 0 "#PWR?" H 5900 5150 50  0001 C CNN
+F 0 "#PWR096" H 5900 5150 50  0001 C CNN
 F 1 "GND" H 5905 5227 50  0000 C CNN
 F 2 "" H 5900 5400 50  0001 C CNN
@@
 AR Path="/5DFD1EC3/5E034394" Ref="#PWR?"  Part="1"
 AR Path="/5E02C61B/5E034394" Ref="#PWR?"  Part="1"
-AR Path="/5E08B2E9/5E034394" Ref="#PWR?"  Part="1"
+AR Path="/5E08B2E9/5E034394" Ref="#PWR092"  Part="1"
 AR Path="/5E0EDFEE/5E034394" Ref="#PWR?"  Part="1"
-F 0 "#PWR?" H 3000 3450 50  0001 C CNN
+F 0 "#PWR092" H 3000 3450 50  0001 C CNN
 F 1 "GND" H 3005 3527 50  0000 C CNN
 F 2 "" H 3000 3700 50  0001 C CNN
@@
 AR Path="/5DFD1EC3/5E0343A3" Ref="Y?"  Part="1"
 AR Path="/5E02C61B/5E0343A3" Ref="Y?"  Part="1"
-AR Path="/5E08B2E9/5E0343A3" Ref="Y?"  Part="1"
+AR Path="/5E08B2E9/5E0343A3" Ref="Y12"  Part="1"
 AR Path="/5E0EDFEE/5E0343A3" Ref="Y?"  Part="1"
-F 0 "Y?" V 3904 3581 50  0000 L CNN
+F 0 "Y12" V 3904 3581 50  0000 L CNN
 F 1 "8MHz" V 3995 3581 50  0000 L CNN
 F 2 "Crystal:Crystal_SMD_3225-4Pin_3.2x2.5mm_HandSoldering" H 3950 3450 50  0001 C CNN
@@
 AR Path="/5DFD1EC3/5E0343AB" Ref="R?"  Part="1"
 AR Path="/5E02C61B/5E0343AB" Ref="R?"  Part="1"
-AR Path="/5E08B2E9/5E0343AB" Ref="R?"  Part="1"
+AR Path="/5E08B2E9/5E0343AB" Ref="R34"  Part="1"
 AR Path="/5E0EDFEE/5E0343AB" Ref="R?"  Part="1"
-F 0 "R?" V 4293 2600 50  0000 C CNN
+F 0 "R34" V 4293 2600 50  0000 C CNN
 F 1 "10K" V 4384 2600 50  0000 C CNN
 F 2 "Resistor_SMD:R_0603_1608Metric" V 4430 2600 50  0001 C CNN
@@
 AR Path="/5DFD1EC3/5E0343B2" Ref="#PWR?"  Part="1"
 AR Path="/5E02C61B/5E0343B2" Ref="#PWR?"  Part="1"
-AR Path="/5E08B2E9/5E0343B2" Ref="#PWR?"  Part="1"
+AR Path="/5E08B2E9/5E0343B2" Ref="#PWR094"  Part="1"
 AR Path="/5E0EDFEE/5E0343B2" Ref="#PWR?"  Part="1"
-F 0 "#PWR?" H 4200 2550 50  0001 C CNN
+F 0 "#PWR094" H 4200 2550 50  0001 C CNN
 F 1 "GND" H 4205 2627 50  0000 C CNN
 F 2 "" H 4200 2800 50  0001 C CNN
@@
 AR Path="/5DFD1EC3/5E0343B8" Ref="#PWR?"  Part="1"
 AR Path="/5E02C61B/5E0343B8" Ref="#PWR?"  Part="1"
-AR Path="/5E08B2E9/5E0343B8" Ref="#PWR?"  Part="1"
+AR Path="/5E08B2E9/5E0343B8" Ref="#PWR093"  Part="1"
 AR Path="/5E0EDFEE/5E0343B8" Ref="#PWR?"  Part="1"
-F 0 "#PWR?" H 3400 4600 50  0001 C CNN
+F 0 "#PWR093" H 3400 4600 50  0001 C CNN
 F 1 "GND" H 3405 4677 50  0000 C CNN
 F 2 "" H 3400 4850 50  0001 C CNN
@@
 AR Path="/5DFD1EC3/5E0343C1" Ref="U?"  Part="1"
 AR Path="/5E02C61B/5E0343C1" Ref="U?"  Part="1"
-AR Path="/5E08B2E9/5E0343C1" Ref="U?"  Part="1"
+AR Path="/5E08B2E9/5E0343C1" Ref="U29"  Part="1"
 AR Path="/5E0EDFEE/5E0343C1" Ref="U?"  Part="1"
-F 0 "U?" H 5450 2311 50  0000 C CNN
+F 0 "U29" H 5450 2311 50  0000 C CNN
 F 1 "STM32F103C8T6" H 5450 2220 50  0000 C CNN
 F 2 "Package_QFP:LQFP-48_7x7mm_P0.5mm" H 4900 2500 50  0001 R CNN
@@
 AR Path="/5E0343D4" Ref="J?"  Part="1"
 AR Path="/5E0EDFEE/5E0343D4" Ref="J?"  Part="1"
-F 0 "J?" H 6780 5042 50  0000 L CNN
+AR Path="/5E08B2E9/5E0343D4" Ref="J12"  Part="1"
+F 0 "J12" H 6780 5042 50  0000 L CNN
 F 1 "Conn_01x03" H 6780 4951 50  0000 L CNN
 F 2 "RuanProject:Connector_Set_1x03_P2.54mm_Vertical" H 6700 5000 50  0001 C CNN
