File: LED_Part12.sch (KiCad schematic (older format))
At the start: 13 parts

Commit message: Ruan: modify LED part
Parts:
- gave numbers to parts that had none: 13
Changed lines of the file:
@@
 AR Path="/5E02C61B/5DD26DDC" Ref="R?"  Part="1"
 AR Path="/5E08B2E9/5DD26DDC" Ref="R?"  Part="1"
-AR Path="/5E0EDFEE/5DD26DDC" Ref="R?"  Part="1"
-F 0 "R?" V 7593 3300 50  0000 C CNN
+AR Path="/5E0EDFEE/5DD26DDC" Ref="R37"  Part="1"
+F 0 "R37" V 7593 3300 50  0000 C CNN
 F 1 "10K" V 7684 3300 50  0000 C CNN
 F 2 "Resistor_SMD:R_0603_1608Metric" V 7730 3300 50  0001 C CNN
@@
 AR Path="/5E02C61B/5DD26E87" Ref="U?"  Part="1"
 AR Path="/5E08B2E9/5DD26E87" Ref="U?"  Part="1"
-AR Path="/5E0EDFEE/5DD26E87" Ref="U?"  Part="1"
-F 0 "U?" H 3800 4215 50  0000 C CNN
+AR Path="/5E0EDFEE/5DD26E87" Ref="U30"  Part="1"
+F 0 "U30" H 3800 4215 50  0000 C CNN
 F 1 "TCS3200" H 3800 4124 50  0000 C CNN
 F 2 "Package_SO:SOIC-8_3.9x4.9mm_P1.27mm" H 3700 3950 50  0001 C CNN
@@
 AR Path="/5E02C61B/5DD26E8E" Ref="C?"  Part="1"
 AR Path="/5E08B2E9/5DD26E8E" Ref="C?"  Part="1"
-AR Path="/5E0EDFEE/5DD26E8E" Ref="C?"  Part="1"
-F 0 "C?" H 4035 4804 50  0000 R CNN
+AR Path="/5E0EDFEE/5DD26E8E" Ref="C96"  Part="1"
+F 0 "C96" H 4035 4804 50  0000 R CNN
 F 1 "0.1uF" H 4035 4895 50  0000 R CNN
 F 2 "Capacitor_SMD:C_0603_1608Metric" H 4188 4700 50  0001 C CNN
@@
 AR Path="/5E02C61B/5DD26E94" Ref="C?"  Part="1"
 AR Path="/5E08B2E9/5DD26E94" Ref="C?"  Part="1"
-AR Path="/5E0EDFEE/5DD26E94" Ref="C?"  Part="1"
-F 0 "C?" V 3452 3150 50  0000 C CNN
+AR Path="/5E0EDFEE/5DD26E94" Ref="C95"  Part="1"
+F 0 "C95" V 3452 3150 50  0000 C CNN
 F 1 "20pF" V 3361 3150 50  0000 C CNN
 F 2 "Capacitor_SMD:C_0603_1608Metric" H 3238 3000 50  0001 C CNN
@@
 AR Path="/5E02C61B/5DD26E9A" Ref="C?"  Part="1"
 AR Path="/5E08B2E9/5DD26E9A" Ref="C?"  Part="1"
-AR Path="/5E0EDFEE/5DD26E9A" Ref="C?"  Part="1"
-F 0 "C?" V 3452 2800 50  0000 C CNN
+AR Path="/5E0EDFEE/5DD26E9A" Ref="C94"  Part="1"
+F 0 "C94" V 3452 2800 50  0000 C CNN
 F 1 "20pF" V 3361 2800 50  0000 C CNN
 F 2 "Capacitor_SMD:C_0603_1608Metric" H 3238 2650 50  0001 C CNN
@@
 AR Path="/5E02C61B/5DD26EA0" Ref="C?"  Part="1"
 AR Path="/5E08B2E9/5DD26EA0" Ref="C?"  Part="1"
-AR Path="/5E0EDFEE/5DD26EA0" Ref="C?"  Part="1"
-F 0 "C?" H 6735 2104 50  0000 R CNN
+AR Path="/5E0EDFEE/5DD26EA0" Ref="C100"  Part="1"
+F 0 "C100" H 6735 2104 50  0000 R CNN
 F 1 "0.1uF" H 6735 2195 50  0000 R CNN
 F 2 "Capacitor_SMD:C_0603_1608Metric" H 6888 2000 50  0001 C CNN
@@
 AR Path="/5E02C61B/5DD26EA8" Ref="C?"  Part="1"
 AR Path="/5E08B2E9/5DD26EA8" Ref="C?"  Part="1"
-AR Path="/5E0EDFEE/5DD26EA8" Ref="C?"  Part="1"
-F 0 "C?" H 6435 2104 50  0000 R CNN
+AR Path="/5E0EDFEE/5DD26EA8" Ref="C99"  Part="1"
+F 0 "C99" H 6435 2104 50  0000 R CNN
 F 1 "0.1uF" H 6435 2195 50  0000 R CNN
 F 2 "Capacitor_SMD:C_0603_1608Metric" H 6588 2000 50  0001 C CNN
@@
 AR Path="/5E02C61B/5DD26EB4" Ref="#PWR?"  Part="1"
 AR Path="/5E08B2E9/5DD26EB4" Ref="#PWR?"  Part="1"
-AR Path="/5E0EDFEE/5DD26EB4" Ref="#PWR?"  Part="1"
-F 0 "#PWR?" H 6400 2250 50  0001 C CNN
+AR Path="/5E0EDFEE/5DD26EB4" Ref="#PWR0105"  Part="1"
+F 0 "#PWR0105" H 6400 2250 50  0001 C CNN
 F 1 "GND" H 6405 2327 50  0000 C CNN
 F 2 "" H 6400 2500 50  0001 C CNN
@@
 AR Path="/5E02C61B/5DD26EBA" Ref="C?"  Part="1"
 AR Path="/5E08B2E9/5DD26EBA" Ref="C?"  Part="1"
-AR Path="/5E0EDFEE/5DD26EBA" Ref="C?"  Part="1"
-F 0 "C?" H 6135 2104 50  0000 R CNN
+AR Path="/5E0EDFEE/5DD26EBA" Ref="C98"  Part="1"
+F 0 "C98" H 6135 2104 50  0000 R CNN
 F 1 "0.1uF" H 6135 2195 50  0000 R CNN
 F 2 "Capacitor_SMD:C_0603_1608Metric" H 6288 2000 50  0001 C CNN
@@
 AR Path="/5E02C61B/5DD26EC0" Ref="C?"  Part="1"
 AR Path="/5E08B2E9/5DD26EC0" Ref="C?"  Part="1"
-AR Path="/5E0EDFEE/5DD26EC0" Ref="C?"  Part="1"
-F 0 "C?" H 5835 2104 50  0000 R CNN
+AR Path="/5E0EDFEE/5DD26EC0" Ref="C97"  Part="1"
+F 0 "C97" H 5835 2104 50  0000 R CNN
 F 1 "1uF" H 5835 2195 50  0000 R CNN
 F 2 "Capacitor_SMD:C_0603_1608Metric" H 5988 2000 50  0001 C CNN
@@
 AR Path="/5E02C61B/5DD26EC7" Ref="#PWR?"  Part="1"
 AR Path="/5E08B2E9/5DD26EC7" Ref="#PWR?"  Part="1"
-AR Path="/5E0EDFEE/5DD26EC7" Ref="#PWR?"  Part="1"
-F 0 "#PWR?" H 6300 4050 50  0001 C CNN
+AR Path="/5E0EDFEE/5DD26EC7" Ref="#PWR0104"  Part="1"
+F 0 "#PWR0104" H 6300 4050 50  0001 C CNN
 F 1 "GND" H 6305 4127 50  0000 C CNN
 F 2 "" H 6300 4300 50  0001 C CNN
@@
 AR Path="/5E02C61B/5DD26EDA" Ref="#PWR?"  Part="1"
 AR Path="/5E08B2E9/5DD26EDA" Ref="#PWR?"  Part="1"
-AR Path="/5E0EDFEE/5DD26EDA" Ref="#PWR?"  Part="1"
-F 0 "#PWR?" H 4150 4750 50  0001 C CNN
+AR Path="/5E0EDFEE/5DD26EDA" Ref="#PWR0102"  Part="1"
+F 0 "#PWR0102" H 4150 4750 50  0001 C CNN
 F 1 "GND" H 4155 4827 50  0000 C CNN
 F 2 "" H 4150 5000 50  0001 C CNN
@@
 AR Path="/5E02C61B/5DD26EF6" Ref="#PWR?"  Part="1"
 AR Path="/5E08B2E9/5DD26EF6" Ref="#PWR?"  Part="1"
-AR Path="/5E0EDFEE/5DD26EF6" Ref="#PWR?"  Part="1"
-F 0 "#PWR?" H 5700 4700 50  0001 C CNN
+AR Path="/5E0EDFEE/5DD26EF6" Ref="#PWR0103"  Part="1"
+F 0 "#PWR0103" H 5700 4700 50  0001 C CNN
 F 1 "GND" H 5705 4777 50  0000 C CNN
 F 2 "" H 5700 4950 50  0001 C CNN
@@
 AR Path="/5E02C61B/5DD26F18" Ref="#PWR?"  Part="1"
 AR Path="/5E08B2E9/5DD26F18" Ref="#PWR?"  Part="1"
-AR Path="/5E0EDFEE/5DD26F18" Ref="#PWR?"  Part="1"
-F 0 "#PWR?" H 2800 3000 50  0001 C CNN
+AR Path="/5E0EDFEE/5DD26F18" Ref="#PWR099"  Part="1"
+F 0 "#PWR099" H 2800 3000 50  0001 C CNN
 F 1 "GND" H 2805 3077 50  0000 C CNN
 F 2 "" H 2800 3250 50  0001 C CNN
@@
 AR Path="/5E02C61B/5DD26F27" Ref="Y?"  Part="1"
 AR Path="/5E08B2E9/5DD26F27" Ref="Y?"  Part="1"
-AR Path="/5E0EDFEE/5DD26F27" Ref="Y?"  Part="1"
-F 0 "Y?" V 3704 3131 50  0000 L CNN
+AR Path="/5E0EDFEE/5DD26F27" Ref="Y13"  Part="1"
+F 0 "Y13" V 3704 3131 50  0000 L CNN
 F 1 "8MHz" V 3795 3131 50  0000 L CNN
 F 2 "Crystal:Crystal_SMD_3225-4Pin_3.2x2.5mm_HandSoldering" H 3750 3000 50  0001 C CNN
@@
 AR Path="/5E02C61B/5DD26F2F" Ref="R?"  Part="1"
 AR Path="/5E08B2E9/5DD26F2F" Ref="R?"  Part="1"
-AR Path="/5E0EDFEE/5DD26F2F" Ref="R?"  Part="1"
-F 0 "R?" V 4093 2150 50  0000 C CNN
+AR Path="/5E0EDFEE/5DD26F2F" Ref="R36"  Part="1"
+F 0 "R36" V 4093 2150 50  0000 C CNN
 F 1 "10K" V 4184 2150 50  0000 C CNN
 F 2 "Resistor_SMD:R_0603_1608Metric" V 4230 2150 50  0001 C CNN
@@
 AR Path="/5E02C61B/5DD26F36" Ref="#PWR?"  Part="1"
 AR Path="/5E08B2E9/5DD26F36" Ref="#PWR?"  Part="1"
-AR Path="/5E0EDFEE/5DD26F36" Ref="#PWR?"  Part="1"
-F 0 "#PWR?" H 4000 2100 50  0001 C CNN
+AR Path="/5E0EDFEE/5DD26F36" Ref="#PWR0101"  Part="1"
+F 0 "#PWR0101" H 4000 2100 50  0001 C CNN
 F 1 "GND" H 4005 2177 50  0000 C CNN
 F 2 "" H 4000 2350 50  0001 C CNN
@@
 AR Path="/5E02C61B/5DD26F3C" Ref="#PWR?"  Part="1"
 AR Path="/5E08B2E9/5DD26F3C" Ref="#PWR?"  Part="1"
-AR Path="/5E0EDFEE/5DD26F3C" Ref="#PWR?"  Part="1"
-F 0 "#PWR?" H 3200 4150 50  0001 C CNN
+AR Path="/5E0EDFEE/5DD26F3C" Ref="#PWR0100"  Part="1"
+F 0 "#PWR0100" H 3200 4150 50  0001 C CNN
 F 1 "GND" H 3205 4227 50  0000 C CNN
 F 2 "" H 3200 4400 50  0001 C CNN
@@
 AR Path="/5E02C61B/5DD26F45" Ref="U?"  Part="1"
 AR Path="/5E08B2E9/5DD26F45" Ref="U?"  Part="1"
-AR Path="/5E0EDFEE/5DD26F45" Ref="U?"  Part="1"
-F 0 "U?" H 5250 1861 50  0000 C CNN
+AR Path="/5E0EDFEE/5DD26F45" Ref="U31"  Part="1"
+F 0 "U31" H 5250 1861 50  0000 C CNN
 F 1 "STM32F103C8T6" H 5250 1770 50  0000 C CNN
 F 2 "Package_QFP:LQFP-48_7x7mm_P0.5mm" H 4700 2050 50  0001 R CNN
@@
 P 6500 4550
 AR Path="/5E02758B" Ref="J?"  Part="1"
-AR Path="/5E0EDFEE/5E02758B" Ref="J?"  Part="1"
-F 0 "J?" H 6580 4592 50  0000 L CNN
+AR Path="/5E0EDFEE/5E02758B" Ref="J13"  Part="1"
+F 0 "J13" H 6580 4592 50  0000 L CNN
 F 1 "Conn_01x03" H 6580 4501 50  0000 L CNN
 F 2 "RuanProject:Connector_Set_1x03_P2.54mm_Vertical" H 6500 4550 50  0001 C CNN
