File: CSWL_Tester_Board.sch (KiCad schematic (older format))
At the start: 74 parts

Commit message: Ruan: modify LED part
Parts:
- removed TP110: TP110, TestPoint:TestPoint_Loop_D2.54mm_Drill1.5mm_Beaded, symbol Connector:TestPoint
- removed TP111: TP111, TestPoint:TestPoint_Loop_D2.54mm_Drill1.5mm_Beaded, symbol Connector:TestPoint
- gave numbers to parts that had none: 40
Connections:
- wire segments 354 -> 351

Commit message: RUan: 12 mcu version
Parts:
- removed J1: Conn_02x32_Counter_Clockwise, symbol Connector_Generic:Conn_02x32_Counter_Clockwise
- added J?: Conn_02x10_Counter_Clockwise, symbol Connector_Generic:Conn_02x10_Counter_Clockwise
Connections:
- wire segments 351 -> 307
Changed lines of the file:
@@
 Text GLabel 7300 4700 2    50   Input ~ 0
 VCC33_D
-$Comp
-L Connector_Generic:Conn_02x32_Counter_Clockwise J1
-U 1 1 5D603B0E
-P 16700 11450
-F 0 "J1" H 16750 13167 50  0000 C CNN
-F 1 "Conn_02x32_Counter_Clockwise" H 16750 13076 50  0000 C CNN
-F 2 "" H 16700 11450 50  0001 C CNN
-F 3 "~" H 16700 11450 50  0001 C CNN
-	1    16700 11450
-	1    0    0    -1
-$EndComp
 Wire Wire Line
 	16000 9950 16500 9950
@@
 	16500 10450 16000 10450
 Wire Wire Line
-	16500 10950 16000 10950
-Wire Wire Line
-	16500 11050 16000 11050
-Wire Wire Line
-	16000 11150 16500 11150
-Wire Wire Line
-	16500 11250 16000 11250
-Wire Wire Line
-	16500 11350 16000 11350
-Wire Wire Line
-	16500 11450 16000 11450
-Wire Wire Line
-	16000 11550 16500 11550
-Wire Wire Line
-	16500 11650 16000 11650
-Wire Wire Line
-	16500 11750 16000 11750
-Wire Wire Line
-	16500 11850 16000 11850
-Wire Wire Line
-	16000 11950 16500 11950
-Wire Wire Line
-	16500 12050 16000 12050
-Wire Wire Line
-	16500 12150 16000 12150
-Wire Wire Line
-	16500 12250 16000 12250
-Wire Wire Line
-	16000 12350 16500 12350
-Wire Wire Line
-	16500 12450 16000 12450
-Wire Wire Line
-	16000 12750 16500 12750
-Wire Wire Line
-	16500 12850 16000 12850
-Wire Wire Line
-	16500 12950 16000 12950
-Wire Wire Line
-	16500 13050 16000 13050
-Wire Wire Line
-	17500 11450 17000 11450
-Wire Wire Line
-	17000 11350 17500 11350
-Wire Wire Line
-	17000 11250 17500 11250
-Wire Wire Line
-	17000 11150 17500 11150
-Wire Wire Line
-	17500 11050 17000 11050
-Wire Wire Line
-	17000 10950 17500 10950
-Wire Wire Line
 	17000 10850 17500 10850
 Wire Wire Line
@@
 Wire Wire Line
 	17000 9950 17500 9950
-Wire Wire Line
-	17500 13050 17000 13050
-Wire Wire Line
-	17000 12950 17500 12950
-Wire Wire Line
-	17000 12850 17500 12850
-Wire Wire Line
-	17000 12750 17500 12750
-Wire Wire Line
-	17500 12650 17000 12650
-Wire Wire Line
-	17000 12550 17500 12550
-Wire Wire Line
-	17000 12450 17500 12450
-Wire Wire Line
-	17000 12350 17500 12350
-Wire Wire Line
-	17500 12250 17000 12250
-Wire Wire Line
-	17000 12150 17500 12150
-Wire Wire Line
-	17000 12050 17500 12050
-Wire Wire Line
-	17000 11950 17500 11950
-Wire Wire Line
-	17500 11850 17000 11850
-Wire Wire Line
-	17000 11750 17500 11750
-Wire Wire Line
-	17000 11650 17500 11650
-Wire Wire Line
-	17000 11550 17500 11550
-Wire Wire Line
-	15850 12550 16500 12550
-Wire Wire Line
-	15850 12650 16500 12650
 Text Label 17100 10050 0    50   ~ 0
 LED_UsartTx
@@
 Text Label 15400 10650 0    50   ~ 0
 CSWL_VDD-
+$Comp
+L Connector_Generic:Conn_02x10_Counter_Clockwise J?
+U 1 1 5D29E733
+P 16700 10350
+F 0 "J?" H 16750 10967 50  0000 C CNN
+F 1 "Conn_02x10_Counter_Clockwise" H 16750 10876 50  0000 C CNN
+F 2 "" H 16700 10350 50  0001 C CNN
+F 3 "~" H 16700 10350 50  0001 C CNN
+	1    16700 10350
+	1    0    0    -1
+$EndComp
 $EndSCHEMATC

Commit message: Ruan: V0
Parts:
- removed C10, C4, C6, C7, C8, C9: 1uF, Capacitor_SMD:C_0603_1608Metric, symbol Device:C
- removed Q1: 2N7002LT1G, digikey-footprints:SOT-23-3, symbol dk_Transistors-FETs-MOSFETs-Single:2N7002LT1G
- removed R1: 33R, Resistor_SMD:R_0603_1608Metric, symbol Device:R
- removed R11, R12, R13, R3, R6, R7, R8, R9: 10K, Resistor_SMD:R_0603_1608Metric, symbol Device:R
- removed R2: 100K, Resistor_SMD:R_0603_1608Metric, symbol Device:R
- removed U4, U5, U6: MCP1700T-3302E_TT, digikey-footprints:SOT-23-3, symbol dk_PMIC-Voltage-Regulators-Linear:MCP1700T-3302E_TT
- added C? (x12): 0.1uF, Capacitor_SMD:C_0603_1608Metric, symbol Device:C
- added C? (x2): 1uF, Capacitor_SMD:C_0603_1608Metric, symbol Device:C
- added D?: LED1, symbol Device:LED
- added D? (x3): LED2, symbol Device:LED
- added D? (x3): LED3, symbol Device:LED
- added D? (x3): LED4, symbol Device:LED
- added D? (x2): LED, symbol Device:LED
- added Q? (x5): 2N7002LT1G, digikey-footprints:SOT-23-3, symbol dk_Transistors-FETs-MOSFETs-Single:2N7002LT1G
- added R? (x83): 10K, Resistor_SMD:R_0603_1608Metric, symbol Device:R
- added R? (x5): 33R, Resistor_SMD:R_0603_1608Metric, symbol Device:R
- added R? (x5): 100K, Resistor_SMD:R_0603_1608Metric, symbol Device:R
- added U? (x9): sn74hc595, Package_SO:SOIC-16_3.9x9.9mm_P1.27mm, symbol 74xx:74HC595
- added U? (x12): TCS3200, Package_SO:SOIC-8_3.9x4.9mm_P1.27mm, symbol RuanProject:TCS3200
- added U? (x2): SN74HC151DR, Package_SO:SOIC-16_3.9x9.9mm_P1.27mm, symbol 74xx:74LS151
- added U?: MCP1700T-3302E_TT, digikey-footprints:SOT-23-3, symbol dk_PMIC-Voltage-Regulators-Linear:MCP1700T-3302E_TT
Connections:
- net labels added: GB10, GB11, GB12, GB13, GB14, GB9, LED1-6_Output, LED10_EN, LED10_OUT, LED10_S0, LED10_S1, LED10_S2, LED10_S3, LED11_EN, LED11_OUT, LED11_S0, LED11_S1, LED11_S2, LED11_S3, LED12_EN, LED12_OUT, LED12_S0, LED12_S1, LED12_S2, LED12_S3, LED1_EN, LED1_OUT, LED1_S0, LED1_S1, LED1_S2, LED1_S3, LED2_EN, LED2_OUT, LED2_S0, LED2_S1, LED2_S2, LED2_S3, LED3_EN, LED3_OUT, LED3_S0, LED3_S1, LED3_S2, LED3_S3, LED4_EN, LED4_OUT, LED4_S0, LED4_S1, LED4_S2, LED4_S3, LED5_EN, LED5_OUT, LED5_S0, LED5_S1, LED5_S2, LED5_S3, LED6_EN, LED6_OUT, LED6_S0, LED6_S1, LED6_S2, LED6_S3, LED7-12_Output, LED7-8_Output, LED7_EN, LED7_OUT, LED7_S0, LED7_S1, LED7_S2, LED7_S3, LED8_EN, LED8_OUT, LED8_S0, LED8_S1, LED8_S2, LED8_S3, LED9_EN, LED9_OUT, LED9_S0, LED9_S1, LED9_S2, LED9_S3, Serial_CLK, Serial_Input, Serial_Ouput, Serial_nEN, Shift_reg_clear, Shift_reg_lock, Switchs_S0, Switchs_S1, Switchs_S2, Switchs_S3
- net labels removed: LED10_ENSS, LED11_ENSS, LED12_ENSS, LED1_ENSS, LED2_ENSS, LED3_ENSS, LED4_ENSS, LED5_ENSS, LED6_ENSS, LED7_ENSS, LED8_ENSS, LED9_ENSS, LED_GPIO0, LED_GPIO1, LED_GPIO2, LED_GPIO3, SPI1_MISO, SPI1_MOSI, SPI1_SCK, VCC33_C, VCC33_D
- wire segments 307 -> 695
- no-connect marks 0 -> 6
Other:
- note removed: "LED capture \n"
- moved on the sheet: C1, C2, C3, C5, J?, R4, R5, TP106, TP107, TP108, TP109, TP110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

Commit message: Ruan: base ok
Parts:
- removed C1, C14, C15, C16, C2, C? (x12): 0.1uF, Capacitor_SMD:C_0603_1608Metric, symbol Device:C
- removed C11, C12: 20pF, Capacitor_SMD:C_0603_1608Metric, symbol Device:C
- removed C13, C3, C5, C? (x2): 1uF, Capacitor_SMD:C_0603_1608Metric, symbol Device:C
- removed D?: LED1, symbol Device:LED
- removed D? (x3): LED2, symbol Device:LED
- removed D? (x3): LED3, symbol Device:LED
- removed D? (x3): LED4, symbol Device:LED
- removed D? (x2): LED, symbol Device:LED
- removed J2: Conn_01x03, RuanProject:Connector_Set_1x03_P2.54mm_Vertical, symbol Connector_Generic:Conn_01x03
- removed J?: Conn_02x10_Counter_Clockwise, symbol Connector_Generic:Conn_02x10_Counter_Clockwise
- removed Q? (x5): 2N7002LT1G, digikey-footprints:SOT-23-3, symbol dk_Transistors-FETs-MOSFETs-Single:2N7002LT1G
- removed R10, R? (x83): 10K, Resistor_SMD:R_0603_1608Metric, symbol Device:R
- removed R4, R5: 0R, Resistor_SMD:R_0603_1608Metric, symbol Device:R
- removed R? (x5): 33R, Resistor_SMD:R_0603_1608Metric, symbol Device:R
- removed R? (x5): 100K, Resistor_SMD:R_0603_1608Metric, symbol Device:R
- removed TP106: TP106, TestPoint:TestPoint_Loop_D2.54mm_Drill1.5mm_Beaded, symbol Connector:TestPoint
- removed U1, U2: CD74HC4067M, Package_SO:SOIC-24W_7.5x15.4mm_P1.27mm, symbol 74xx:CD74HC4067M
- removed U3, U?: MCP1700T-3302E_TT, digikey-footprints:SOT-23-3, symbol dk_PMIC-Voltage-Regulators-Linear:MCP1700T-3302E_TT
- removed U7: STM32F103C8Tx, Package_QFP:LQFP-48_7x7mm_P0.5mm, symbol MCU_ST_STM32F1:STM32F103C8Tx
- removed U? (x9): sn74hc595, Package_SO:SOIC-16_3.9x9.9mm_P1.27mm, symbol 74xx:74HC595
- removed U? (x12): TCS3200, Package_SO:SOIC-8_3.9x4.9mm_P1.27mm, symbol RuanProject:TCS3200
- removed U? (x2): SN74HC151DR, Package_SO:SOIC-16_3.9x9.9mm_P1.27mm, symbol 74xx:74LS151
- removed Y1: 8MHz, Crystal:Crystal_SMD_3225-4Pin_3.2x2.5mm_HandSoldering, symbol Device:Crystal
- added J1, J2: Conn_02x10_Odd_Even, Connector_IDC:IDC-Header_2x10_P2.54mm_Vertical, symbol Connector_Generic:Conn_02x10_Odd_Even
- added TP1, TP2, TP3, TP300, TP303, TP306: TP, CSWL_Tester_Pin_Board:PinCard_Hole_D2.3mm_1.3dill, symbol Connector:TestPoint
- TP107: value TP107 -> TP; footprint TestPoint:TestPoint_Loop_D2.54mm_Drill1.5mm_Beaded -> CSWL_Tester_Pin_Board:PinCard_Hole_D2.3mm_1.3dill
- TP108, TP109, TP110, TP111, TP200, TP201: footprint TestPoint:TestPoint_Loop_D2.54mm_Drill1.5mm_Beaded -> CSWL_Tester_Pin_Board:PinCard_Hole_D2.3mm_1.3dill
- TP301: value TP301 -> TP; footprint TestPoint:TestPoint_Loop_D2.54mm_Drill1.5mm_Beaded -> CSWL_Tester_Pin_Board:PinCard_Hole_D2.3mm_1.3dill
- TP302: value TP302 -> TP; footprint TestPoint:TestPoint_Loop_D2.54mm_Drill1.5mm_Beaded -> CSWL_Tester_Pin_Board:PinCard_Hole_D2.3mm_1.3dill
- TP304: value TP304 -> TP; footprint TestPoint:TestPoint_Loop_D2.54mm_Drill1.5mm_Beaded -> CSWL_Tester_Pin_Board:PinCard_Hole_D2.3mm_1.3dill
- TP305: value TP305 -> TP; footprint TestPoint:TestPoint_Loop_D2.54mm_Drill1.5mm_Beaded -> CSWL_Tester_Pin_Board:PinCard_Hole_D2.3mm_1.3dill
- TP307: value TP307 -> TP; footprint TestPoint:TestPoint_Loop_D2.54mm_Drill1.5mm_Beaded -> CSWL_Tester_Pin_Board:PinCard_Hole_D2.3mm_1.3dill
- TP308: value TP308 -> TP; footprint TestPoint:TestPoint_Loop_D2.54mm_Drill1.5mm_Beaded -> CSWL_Tester_Pin_Board:PinCard_Hole_D2.3mm_1.3dill
- TP310: value TP310 -> TP; footprint TestPoint:TestPoint_Loop_D2.54mm_Drill1.5mm_Beaded -> CSWL_Tester_Pin_Board:PinCard_Hole_D2.3mm_1.3dill
- TP311: value TP311 -> TP; footprint TestPoint:TestPoint_Loop_D2.54mm_Drill1.5mm_Beaded -> CSWL_Tester_Pin_Board:PinCard_Hole_D2.3mm_1.3dill
- TP313: value TP313 -> TP; footprint TestPoint:TestPoint_Loop_D2.54mm_Drill1.5mm_Beaded -> CSWL_Tester_Pin_Board:PinCard_Hole_D2.3mm_1.3dill
- TP314: value TP314 -> TP; footprint TestPoint:TestPoint_Loop_D2.54mm_Drill1.5mm_Beaded -> CSWL_Tester_Pin_Board:PinCard_Hole_D2.3mm_1.3dill
- TP316: value TP316 -> TP; footprint TestPoint:TestPoint_Loop_D2.54mm_Drill1.5mm_Beaded -> CSWL_Tester_Pin_Board:PinCard_Hole_D2.3mm_1.3dill
- TP317: value TP317 -> TP; footprint TestPoint:TestPoint_Loop_D2.54mm_Drill1.5mm_Beaded -> CSWL_Tester_Pin_Board:PinCard_Hole_D2.3mm_1.3dill
- TP319: value TP319 -> TP; footprint TestPoint:TestPoint_Loop_D2.54mm_Drill1.5mm_Beaded -> CSWL_Tester_Pin_Board:PinCard_Hole_D2.3mm_1.3dill
- TP320: value TP320 -> TP; footprint TestPoint:TestPoint_Loop_D2.54mm_Drill1.5mm_Beaded -> CSWL_Tester_Pin_Board:PinCard_Hole_D2.3mm_1.3dill
- TP322: value TP322 -> TP; footprint TestPoint:TestPoint_Loop_D2.54mm_Drill1.5mm_Beaded -> CSWL_Tester_Pin_Board:PinCard_Hole_D2.3mm_1.3dill
- TP323: value TP323 -> TP; footprint TestPoint:TestPoint_Loop_D2.54mm_Drill1.5mm_Beaded -> CSWL_Tester_Pin_Board:PinCard_Hole_D2.3mm_1.3dill
- TP325: value TP325 -> TP; footprint TestPoint:TestPoint_Loop_D2.54mm_Drill1.5mm_Beaded -> CSWL_Tester_Pin_Board:PinCard_Hole_D2.3mm_1.3dill
- TP326: value TP326 -> TP; footprint TestPoint:TestPoint_Loop_D2.54mm_Drill1.5mm_Beaded -> CSWL_Tester_Pin_Board:PinCard_Hole_D2.3mm_1.3dill
- TP328: value TP328 -> TP; footprint TestPoint:TestPoint_Loop_D2.54mm_Drill1.5mm_Beaded -> CSWL_Tester_Pin_Board:PinCard_Hole_D2.3mm_1.3dill
- TP329: value TP329 -> TP; footprint TestPoint:TestPoint_Loop_D2.54mm_Drill1.5mm_Beaded -> CSWL_Tester_Pin_Board:PinCard_Hole_D2.3mm_1.3dill
- TP331: value TP331 -> TP; footprint TestPoint:TestPoint_Loop_D2.54mm_Drill1.5mm_Beaded -> CSWL_Tester_Pin_Board:PinCard_Hole_D2.3mm_1.3dill
- TP332: value TP332 -> TP; footprint TestPoint:TestPoint_Loop_D2.54mm_Drill1.5mm_Beaded -> CSWL_Tester_Pin_Board:PinCard_Hole_D2.3mm_1.3dill
- TP334: value TP334 -> TP; footprint TestPoint:TestPoint_Loop_D2.54mm_Drill1.5mm_Beaded -> CSWL_Tester_Pin_Board:PinCard_Hole_D2.3mm_1.3dill
- TP335: value TP335 -> TP; footprint TestPoint:TestPoint_Loop_D2.54mm_Drill1.5mm_Beaded -> CSWL_Tester_Pin_Board:PinCard_Hole_D2.3mm_1.3dill
Connections:
- net labels added: AS4_Y, AS4_Z, TP300, TP303, TP306, TPXXX
- net labels removed: +5V, EN, GB10, GB11, GB12, GB13, GB14, GB9, GND, LED1-6_Output, LED10_EN, LED10_OUT, LED10_S0, LED10_S1, LED10_S2, LED10_S3, LED11_EN, LED11_OUT, LED11_S0, LED11_S1, LED11_S2, LED11_S3, LED12_EN, LED12_OUT, LED12_S0, LED12_S1, LED12_S2, LED12_S3, LED1_EN, LED1_OUT, LED1_S0, LED1_S1, LED1_S2, LED1_S3, LED2_EN, LED2_OUT, LED2_S0, LED2_S1, LED2_S2, LED2_S3, LED3_EN, LED3_OUT, LED3_S0, LED3_S1, LED3_S2, LED3_S3, LED4_EN, LED4_OUT, LED4_S0, LED4_S1, LED4_S2, LED4_S3, LED5_EN, LED5_OUT, LED5_S0, LED5_S1, LED5_S2, LED5_S3, LED6_EN, LED6_OUT, LED6_S0, LED6_S1, LED6_S2, LED6_S3, LED7-12_Output, LED7-8_Output, LED7_EN, LED7_OUT, LED7_S0, LED7_S1, LED7_S2, LED7_S3, LED8_EN, LED8_OUT, LED8_S0, LED8_S1, LED8_S2, LED8_S3, LED9_EN, LED9_OUT, LED9_S0, LED9_S1, LED9_S2, LED9_S3, LED_UsartRx, LED_UsartTx, S0, S1, S2, S3, SWDCLK, SWDIO, Serial_CLK, Serial_Input, Serial_Ouput, Serial_nEN, Shift_reg_clear, Shift_reg_lock, Switchs_EN, Switchs_S0, Switchs_S1, Switchs_S2, Switchs_S3, VCC33_A, VCC33_B, VMeter+, VMeter-
- wire segments 695 -> 59
- no-connect marks 6 -> 0
Other:
- note removed: "LED Board\n"
- note removed: "To MainBoard --- Connector\n"
- note removed: "Voltage_measure_path\n\n"
