File: PD_Charging_Power_PCB.sch (KiCad schematic (older format))
At the start: 34 parts, among them J1 105450-0101, Q1 CJQ4459, Q2 2N7002KDW, U1 STUSB4500

Commit message: Ruan: base ok V0.1
Parts:
- removed J1: 105450-0101, RuanProject:MOLEX_105450-0101_modifyed, symbol RuanProject:105450-0101
- added J1: 105450-0101, RuanProject:MOLEX_105450-0101, symbol 105450-0101:105450-0101
- CLK1, INT1, RST1, SDA1, VBUS1: footprint TestPoint:TestPoint_Pad_D1.5mm -> TestPoint:TestPoint_Pad_D1.0mm
- GND1: renamed from TP1; footprint TestPoint:TestPoint_Pad_D1.5mm -> TestPoint:TestPoint_Pad_D1.0mm
- Q2: footprint digikey-footprints:SOT-363 -> RuanProject:SOT-363_SC-70-6
Connections:
- wire segments 133 -> 134
- no-connect marks 11 -> 16
Changed lines of the file:
@@
 F 0 "Q2" H 9000 5437 60  0000 C CNN
 F 1 "2N7002KDW" H 9000 5331 60  0000 C CNN
-F 2 "digikey-footprints:SOT-363" H 9200 5150 60  0001 L CNN
+F 2 "RuanProject:SOT-363_SC-70-6" H 9200 5150 60  0001 L CNN
 F 3 "" H 9200 5250 60  0001 L CNN
 F 4 "MOSFET 2N-CH 60V 300mA VGS = 4.5V, ID =200mA , SOT363" H 9200 5950 60  0001 L CNN "Detail"
@@
 F 0 "CLK1" V 7100 5088 50  0001 L CNN
 F 1 "CLK" V 7145 5088 50  0000 L CNN
-F 2 "TestPoint:TestPoint_Pad_D1.5mm" H 7300 4900 50  0001 C CNN
+F 2 "TestPoint:TestPoint_Pad_D1.0mm" H 7300 4900 50  0001 C CNN
 F 3 "~" H 7300 4900 50  0001 C CNN
 	1    7100 4900
@@
 F 0 "SDA1" V 7100 5238 50  0001 L CNN
 F 1 "SDA" V 7145 5238 50  0000 L CNN
-F 2 "TestPoint:TestPoint_Pad_D1.5mm" H 7300 5050 50  0001 C CNN
+F 2 "TestPoint:TestPoint_Pad_D1.0mm" H 7300 5050 50  0001 C CNN
 F 3 "~" H 7300 5050 50  0001 C CNN
 	1    7100 5050
@@
 F 0 "INT1" V 7100 5338 50  0001 L CNN
 F 1 "INT" V 7145 5338 50  0000 L CNN
-F 2 "TestPoint:TestPoint_Pad_D1.5mm" H 7300 5150 50  0001 C CNN
+F 2 "TestPoint:TestPoint_Pad_D1.0mm" H 7300 5150 50  0001 C CNN
 F 3 "~" H 7300 5150 50  0001 C CNN
 	1    7100 5150
@@
 F 0 "RST1" V 7100 5438 50  0001 L CNN
 F 1 "RST" V 7145 5438 50  0000 L CNN
-F 2 "TestPoint:TestPoint_Pad_D1.5mm" H 7300 5250 50  0001 C CNN
+F 2 "TestPoint:TestPoint_Pad_D1.0mm" H 7300 5250 50  0001 C CNN
 F 3 "~" H 7300 5250 50  0001 C CNN
 	1    7100 5250
@@
 F 0 "VBUS1" V 3500 1238 50  0001 L CNN
 F 1 "VBUS" V 3545 1238 50  0000 L CNN
-F 2 "TestPoint:TestPoint_Pad_D1.5mm" H 3700 1050 50  0001 C CNN
+F 2 "TestPoint:TestPoint_Pad_D1.0mm" H 3700 1050 50  0001 C CNN
 F 3 "~" H 3700 1050 50  0001 C CNN
 	1    3500 1050
@@
 Wire Wire Line
 	3500 2900 3650 2900
-Wire Wire Line
-	3500 2800 3500 2900
-$Comp
-L RuanProject:105450-0101 J1
-U 1 1 5D1785D5
+Connection ~ 3500 1600
+$Comp
+L Connector:TestPoint GND1
+U 1 1 5D1E44D4
+P 3650 2900
+F 0 "GND1" V 3650 3088 50  0001 L CNN
+F 1 "GND" V 3695 3088 50  0000 L CNN
+F 2 "TestPoint:TestPoint_Pad_D1.0mm" H 3850 2900 50  0001 C CNN
+F 3 "~" H 3850 2900 50  0001 C CNN
+	1    3650 2900
+	1    0    0    -1
+$EndComp
+Connection ~ 3650 2900
+Wire Wire Line
+	3650 2900 3750 2900
+$Comp
+L 105450-0101:105450-0101 J1
+U 1 1 5D7A7D47
 P 2800 2300
 F 0 "J1" H 2800 3267 50  0000 C CNN
 F 1 "105450-0101" H 2800 3176 50  0000 C CNN
-F 2 "RuanProject:MOLEX_105450-0101_modifyed" H 2800 2300 50  0001 L BNN
+F 2 "RuanProject:MOLEX_105450-0101" H 2800 2300 50  0001 L BNN
 F 3 "" H 2800 2300 50  0001 L BNN
-F 4 "1054500101" H 2800 2300 50  0001 L BNN "Field4"
-F 5 "None" H 2800 2300 50  0001 L BNN "Field5"
-F 6 "USB Shielded I/O Receptacle; Type C; Right Angle; Surface Mount; Gold over Nickel" H 2800 2300 50  0001 L BNN "Field6"
-F 7 "Molex" H 2800 2300 50  0001 L BNN "Field7"
-F 8 "WM12856CT-ND" H 2800 2300 50  0001 L BNN "Field8"
+F 4 "1054500101" H 2800 2300 50  0001 L BNN "字段4"
+F 5 "None" H 2800 2300 50  0001 L BNN "字段5"
+F 6 "USB Shielded I/O Receptacle; Type C; Right Angle; Surface Mount; Gold over Nickel" H 2800 2300 50  0001 L BNN "字段6"
+F 7 "Molex" H 2800 2300 50  0001 L BNN "字段7"
+F 8 "WM12856CT-ND" H 2800 2300 50  0001 L BNN "字段8"
 	1    2800 2300
 	1    0    0    -1
 $EndComp
-Connection ~ 3500 1600
+Wire Wire Line
+	3500 2800 3500 2900
+Wire Wire Line
+	3500 1800 3500 1900
 Connection ~ 3500 2900
+NoConn ~ 2100 2400
+NoConn ~ 3500 2400
+NoConn ~ 3500 2300
+NoConn ~ 3500 2200
+NoConn ~ 3500 2100
+Wire Wire Line
+	3500 1800 3500 1700
+Connection ~ 3500 1800
+Connection ~ 3500 1700
+Wire Wire Line
+	3500 1700 3500 1600
 Wire Wire Line
 	3500 2600 3500 2700
+Connection ~ 3500 2700
+Wire Wire Line
+	3500 2700 3500 2800
 Connection ~ 3500 2800
-Connection ~ 3500 2700
-Wire Wire Line
-	3500 2700 3500 2800
-Wire Wire Line
-	3500 1600 3500 1700
-Connection ~ 3500 1700
-Wire Wire Line
-	3500 1700 3500 1800
-Connection ~ 3500 1800
-Wire Wire Line
-	3500 1800 3500 1900
-$Comp
-L Connector:TestPoint TP1
-U 1 1 5D1E44D4
-P 3650 2900
-F 0 "TP1" V 3650 3088 50  0001 L CNN
-F 1 "GND" V 3695 3088 50  0000 L CNN
-F 2 "TestPoint:TestPoint_Pad_D1.5mm" H 3850 2900 50  0001 C CNN
-F 3 "~" H 3850 2900 50  0001 C CNN
-	1    3650 2900
-	1    0    0    -1
-$EndComp
-Connection ~ 3650 2900
-Wire Wire Line
-	3650 2900 3750 2900
+Wire Wire Line
+	3500 3000 3500 2900
 $EndSCHEMATC

Commit message: Ruan: update to V0.2
Parts:
- removed TP8: Power Soldering Pad, TestPoint:TestPoint_2Pads_Pitch5.08mm_Drill1.3mm, symbol Connector:TestPoint_2Pole
- added VOUT+1: VOUT+, RuanProject:TestPoint_Pad_4mmx3mm, symbol Connector:TestPoint
- added Vout-1: Vout-, RuanProject:TestPoint_Pad_4mmx3mm, symbol Connector:TestPoint
Connections:
- net GND: now also Vout-1.1
- net at C6.1, D4.2 (A), Q1.5 (D)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: now also VOUT+1.1
Changed lines of the file:
@@
-$EndComp
-$Comp
-L Connector:TestPoint_2Pole TP8
-U 1 1 5CF1B4D0
-P 10350 1600
-F 0 "TP8" H 10350 1795 50  0000 C CNN
-F 1 "Power Soldering Pad" H 10350 1704 50  0000 C CNN
-F 2 "TestPoint:TestPoint_2Pads_Pitch5.08mm_Drill1.3mm" H 10350 1600 50  0001 C CNN
-F 3 "~" H 10350 1600 50  0001 C CNN
-	1    10350 1600
-	1    0    0    -1
 $EndComp
 $Comp
@@
 Wire Wire Line
 	3500 3000 3500 2900
+$Comp
+L Connector:TestPoint VOUT+1
+U 1 1 5D7F5188
+P 10150 1600
+F 0 "VOUT+1" V 10150 1788 50  0001 L CNN
+F 1 "VOUT+" V 10195 1788 50  0000 L CNN
+F 2 "RuanProject:TestPoint_Pad_4mmx3mm" H 10350 1600 50  0001 C CNN
+F 3 "~" H 10350 1600 50  0001 C CNN
+	1    10150 1600
+	1    0    0    -1
+$EndComp
+$Comp
+L Connector:TestPoint Vout-1
+U 1 1 5D7F59F7
+P 10550 1600
+F 0 "Vout-1" V 10550 1788 50  0001 L CNN
+F 1 "Vout-" V 10595 1788 50  0000 L CNN
+F 2 "RuanProject:TestPoint_Pad_4mmx3mm" H 10750 1600 50  0001 C CNN
+F 3 "~" H 10750 1600 50  0001 C CNN
+	1    10550 1600
+	1    0    0    -1
+$EndComp
 $EndSCHEMATC

Commit message: Ruan: V0.3
Parts:
- removed ABS1: ABS, TestPoint:TestPoint_Pad_D1.0mm, symbol Connector:TestPoint
- removed Att1: ATT, TestPoint:TestPoint_Pad_D1.0mm, symbol Connector:TestPoint
- removed C2: 1uF, Capacitor_SMD:C_0603_1608Metric, symbol Device:C
- removed D3: BAT54W, Package_TO_SOT_SMD:SOT-323_SC-70, symbol Diode:BAT54W
- removed R1: 470R, Resistor_SMD:R_0603_1608Metric, symbol Device:R
- C1: footprint Capacitor_SMD:C_1206_3216Metric -> Capacitor_SMD:C_0603_1608Metric; Detail 4.7 µF CAPC3216N X7R 25 V ±20% 1206 -> Auto CAP CER 4.7uF 25V 10% X5R 0603; PN (none) -> Murata GRT188R61E475KE13D; 字段4 (none) -> TDK C1608X5R1E475K080AC
- C3, C4, C5: footprint Capacitor_SMD:C_0603_1608Metric -> Capacitor_SMD:C_0402_1005Metric; Detail 1 µF CAPC1608N X5R 25 V ±20% 0603 -> CAP CER 1UF 25V X5R 0402 10%; PN (none) -> Murata GRT155R61E105KE01D
- C6: footprint Capacitor_SMD:C_0603_1608Metric -> Capacitor_SMD:C_0402_1005Metric; Detail 100 nF CAPC1608N X7R 50 V ±10% 0603 -> CAP CER 0.1UF 50V X7R 0402 10%; PN (none) -> Murata GCM155R71H104KE02D
- D1: value ESD24VC2 -> ESDA25W; footprint Package_TO_SOT_SMD:SOT-23 -> Package_TO_SOT_SMD:SOT-323_SC-70; PN (none) -> ST ESDA25W
- D2, D4: PN (none) -> ST ESDA25P35-1U1M
- J1: Detail (none) -> CONN RCP USB3.1 TYPEC 24P SMD RA; PN (none) -> MOLEX 105450-0101
- Q1: value CJQ4459 -> STL6P3LLH6; footprint RuanProject:SOP-8_CJQ4459 -> RuanProject:PowerFLAT-3x3mm-8pin; Detail (none) -> MOSFET P-CH 30V 6A POWERFLAT; PN (none) -> ST STL6P3LLH6
- Q2: PN (none) -> JCET 2N7002KDW
- R10: footprint Resistor_SMD:R_0603_1608Metric -> Resistor_SMD:R_0402_1005Metric; Detail 100 RESC1608N ±5% 0603 SMD -> RES 100 OHM 5% 1/10W 0402; PN (none) -> KOA RK73B1ETTP101J
- R11, R2: Detail 1 k RESC1608N ±1% 0603 SMD -> RES 1K OHM 5% 1/8W 0603; PN (none) -> KOA RK73B1JTTD102J
- R3, R6: footprint Resistor_SMD:R_0603_1608Metric -> Resistor_SMD:R_0402_1005Metric; Detail 100 k RESC1608N ±5% 0603 SMD -> RES 100K OHM 1% 1/10W 0402; PN (none) -> KOA RK73H1ETTP1003F
- R4, R5: Detail 0R 0402 SMD -> RES 0 OHM JUMPER 0402; PN (none) -> KOA RK73Z1ETTP
- R7: footprint Resistor_SMD:R_0603_1608Metric -> Resistor_SMD:R_0402_1005Metric; Detail 22k RESC1608N ±5% 0603 SMD -> RES 22K OHM 5% 1/10W 0402; PN (none) -> KOA RK73B1ETTP223J
- R8, R9: Detail 10 k ±5% 0402 SMD -> RES, 1/10W, 1%, 0402, SMD, 10k; PN (none) -> KOA RK73H1ETTP1002F
- U1: Detail (none) -> IC USB CONTROLLER I2C 24QFN; PN (none) -> ST STUSB4500QTR
- renumbered VOUT+1 to VOUT1, Vout-1 to Vout2
Connections:
- net VBUS: now also R2.1

Commit message: Ruan: change to V0.5
Parts:
- added D3: Power_LED, RuanProject:Led-LTST-S270KGKT, symbol Device:LED
- added R1: 2.2K, Resistor_SMD:R_0402_1005Metric, symbol Device:R
- R4: value 0R(NC) -> 0R (NC)
- R5: value 0R(NC) -> 0R
Connections:
- net GND: now also D3.1 (K)
- net at C6.1, D4.2 (A), Q1.5 (D)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: now also R1.2
- new net: D3.2 (A), R1.1
Changed lines of the file:
@@
 Connection ~ 7750 2200
-Wire Wire Line
-	7750 2500 7750 4000
 Wire Wire Line
 	7750 2200 8100 2200
@@
 	9300 5350 9350 5350
 $Comp
-L Device:R R8
-U 1 1 5CF66D6E
-P 7750 5150
-F 0 "R8" H 7820 5196 50  0000 L CNN
-F 1 "10K" H 7820 5105 50  0000 L CNN
-F 2 "Resistor_SMD:R_0402_1005Metric" V 7680 5150 50  0001 C CNN
-F 3 "~" H 7750 5150 50  0001 C CNN
-F 4 "RES, 1/10W, 1%, 0402, SMD, 10k" H 7750 5150 50  0001 C CNN "Detail"
-F 5 "KOA RK73H1ETTP1002F" H 7750 5150 50  0001 C CNN "PN"
-	1    7750 5150
-	1    0    0    -1
-$EndComp
-$Comp
-L Device:R R9
-U 1 1 5CF67317
-P 8100 4950
-F 0 "R9" H 8170 4996 50  0000 L CNN
-F 1 "10K" H 8170 4905 50  0000 L CNN
-F 2 "Resistor_SMD:R_0402_1005Metric" V 8030 4950 50  0001 C CNN
-F 3 "~" H 8100 4950 50  0001 C CNN
-F 4 "RES, 1/10W, 1%, 0402, SMD, 10k" H 8100 4950 50  0001 C CNN "Detail"
-F 5 "KOA RK73H1ETTP1002F" H 8100 4950 50  0001 C CNN "PN"
-	1    8100 4950
-	1    0    0    -1
-$EndComp
-$Comp
 L power:+2V8 #PWR011
 U 1 1 5CF67C4D
@@
 NoConn ~ 6900 4200
 $Comp
-L Device:R R5
-U 1 1 5D072A33
-P 7300 4350
-F 0 "R5" V 7200 4200 50  0000 L CNN
-F 1 "0R(NC)" V 7200 4350 50  0000 L CNN
-F 2 "Resistor_SMD:R_0402_1005Metric" V 7230 4350 50  0001 C CNN
-F 3 "~" H 7300 4350 50  0001 C CNN
-F 4 "RES 0 OHM JUMPER 0402" H 7300 4350 50  0001 C CNN "Detail"
-F 5 "KOA RK73Z1ETTP" H 7300 4350 50  0001 C CNN "PN"
-	1    7300 4350
-	0    1    1    0
-$EndComp
-$Comp
 L Connector:TestPoint VBUS1
 U 1 1 5D07C1AD
@@
 Wire Wire Line
 	3500 1050 3500 950
-$Comp
-L Device:R R4
-U 1 1 5D0918C3
-P 7300 4000
-F 0 "R4" V 7150 3900 50  0000 L CNN
-F 1 "0R(NC)" V 7150 4050 50  0000 L CNN
-F 2 "Resistor_SMD:R_0402_1005Metric" V 7230 4000 50  0001 C CNN
-F 3 "~" H 7300 4000 50  0001 C CNN
-F 4 "RES 0 OHM JUMPER 0402" H 7300 4000 50  0001 C CNN "Detail"
-F 5 "KOA RK73Z1ETTP" H 7300 4000 50  0001 C CNN "PN"
-	1    7300 4000
-	0    1    1    0
-$EndComp
-Wire Wire Line
-	9150 1600 10000 1600
 Connection ~ 9150 1600
 Connection ~ 10000 1600
 Wire Wire Line
-	6900 4000 7150 4000
-Wire Wire Line
-	7450 4000 7750 4000
-Connection ~ 7750 4000
-Wire Wire Line
 	6900 4350 7150 4350
 Wire Wire Line
-	7450 4350 7750 4350
-Wire Wire Line
-	7750 4350 7750 4000
-Connection ~ 7750 4350
-Wire Wire Line
 	9350 4350 9350 4750
-Wire Wire Line
-	7750 4350 9350 4350
 Wire Wire Line
 	6900 4100 8100 4100
@@
 Wire Wire Line
 	4900 1600 4900 2300
+$Comp
+L Device:LED D3
+U 1 1 5DFD0754
+P 9540 2670
+F 0 "D3" V 9579 2552 50  0000 R CNN
+F 1 "Power_LED" V 9488 2552 50  0000 R CNN
+F 2 "RuanProject:Led-LTST-S270KGKT" H 9540 2670 50  0001 C CNN
+F 3 "~" H 9540 2670 50  0001 C CNN
+F 4 "Lite-On LTST-S270KGKT" V 9540 2670 50  0001 C CNN "PN"
+	1    9540 2670
+	0    -1   -1   0
+$EndComp
+Wire Wire Line
+	7750 4350 9350 4350
+Wire Wire Line
+	7450 4350 7750 4350
+Connection ~ 7750 4350
+Wire Wire Line
+	7750 2500 7750 4000
+Wire Wire Line
+	6900 4000 7150 4000
+$Comp
+L Device:R R5
+U 1 1 5D072A33
+P 7300 4350
+F 0 "R5" V 7190 4210 50  0000 L CNN
+F 1 "0R" V 7200 4370 50  0000 L CNN
+F 2 "Resistor_SMD:R_0402_1005Metric" V 7230 4350 50  0001 C CNN
+F 3 "~" H 7300 4350 50  0001 C CNN
+F 4 "RES 0 OHM JUMPER 0402" H 7300 4350 50  0001 C CNN "Detail"
+F 5 "KOA RK73Z1ETTP" H 7300 4350 50  0001 C CNN "PN"
+	1    7300 4350
+	0    1    1    0
+$EndComp
+$Comp
+L Device:R R9
+U 1 1 5CF67317
+P 8100 4950
+F 0 "R9" H 8170 4996 50  0000 L CNN
+F 1 "10K" H 8170 4905 50  0000 L CNN
+F 2 "Resistor_SMD:R_0402_1005Metric" V 8030 4950 50  0001 C CNN
+F 3 "~" H 8100 4950 50  0001 C CNN
+F 4 "RES, 1/10W, 1%, 0402, SMD, 10k" H 8100 4950 50  0001 C CNN "Detail"
+F 5 "KOA RK73H1ETTP1002F" H 8100 4950 50  0001 C CNN "PN"
+	1    8100 4950
+	1    0    0    -1
+$EndComp
+Wire Wire Line
+	7450 4000 7750 4000
+Connection ~ 7750 4000
+Wire Wire Line
+	7750 4000 7750 4350
+$Comp
+L Device:R R4
+U 1 1 5DFEB544
+P 7300 4000
+F 0 "R4" V 7200 3850 50  0000 L CNN
+F 1 "0R (NC)" V 7200 4000 50  0000 L CNN
+F 2 "Resistor_SMD:R_0402_1005Metric" V 7230 4000 50  0001 C CNN
+F 3 "~" H 7300 4000 50  0001 C CNN
+F 4 "RES 0 OHM JUMPER 0402" H 7300 4000 50  0001 C CNN "Detail"
+F 5 "KOA RK73Z1ETTP" H 7300 4000 50  0001 C CNN "PN"
+	1    7300 4000
+	0    1    1    0
+$EndComp
+Wire Wire Line
+	9540 2360 9540 2520
+Wire Wire Line
+	9540 2820 9540 3000
+$Comp
+L power:GND #PWR0101
+U 1 1 5DFFAF6A
+P 9540 3000
+F 0 "#PWR0101" H 9540 2750 50  0001 C CNN
+F 1 "GND" H 9545 2827 50  0000 C CNN
+F 2 "" H 9540 3000 50  0001 C CNN
+F 3 "" H 9540 3000 50  0001 C CNN
+	1    9540 3000
+	1    0    0    -1
+$EndComp
+Wire Wire Line
+	9150 1600 9540 1600
+$Comp
+L Device:R R1
+U 1 1 5DFE1EBF
+P 9540 2210
+F 0 "R1" V 9478 1993 50  0000 L CNN
+F 1 "2.2K" V 9439 2129 50  0000 L CNN
+F 2 "Resistor_SMD:R_0402_1005Metric" V 9470 2210 50  0001 C CNN
+F 3 "~" H 9540 2210 50  0001 C CNN
+F 4 "RES 2.2K OHM 0402" H 9540 2210 50  0001 C CNN "Detail"
+F 5 "KOA RK73B1ETTP222J" H 9540 2210 50  0001 C CNN "PN"
+	1    9540 2210
+	-1   0    0    1
+$EndComp
+Wire Wire Line
+	9540 2060 9540 1600
+Connection ~ 9540 1600
+Wire Wire Line
+	9540 1600 10000 1600
+$Comp
+L Device:R R8
+U 1 1 5CF66D6E
+P 7750 5150
+F 0 "R8" H 7820 5196 50  0000 L CNN
+F 1 "10K" H 7820 5105 50  0000 L CNN
+F 2 "Resistor_SMD:R_0402_1005Metric" V 7680 5150 50  0001 C CNN
+F 3 "~" H 7750 5150 50  0001 C CNN
+F 4 "RES, 1/10W, 1%, 0402, SMD, 10k" H 7750 5150 50  0001 C CNN "Detail"
+F 5 "KOA RK73H1ETTP1002F" H 7750 5150 50  0001 C CNN "PN"
+	1    7750 5150
+	1    0    0    -1
+$EndComp
 $EndSCHEMATC
